Commit message: sick changes

File: urdf/sick_tim.urdf.xacro (robot description, xacro)
@@ -36,6 +36,6 @@
           <mesh filename="${mesh}" />
         </geometry>
-        <material name="blue" >
-          <color rgba="0 0 1 1" />
+        <material name="gray" >
+          <color rgba="0.7 0.7 0.6 1" />
         </material>
       </visual>
